Commit message: new branch

File: description/urdf/robot_base.urdf (robot description, URDF)
Before this commit: robot None, 1 links, 0 joints
Links:
- added link caster_wheel, mass 0.5; collision sphere radius=0.05; visual sphere radius=0.05
- added link left_wheel, mass 0.8; collision cylinder length=0.04 radius=0.05; visual cylinder length=0.04 radius=0.05
- added link right_wheel, mass 0.8; collision cylinder length=0.04 radius=0.05; visual cylinder length=0.04 radius=0.05
- link base_link: mass None -> 4.2; geometry collision box size=0.4 0.25 0.15; visual box size=0.4 0.25 0.15
Joints:
- added joint connection_link: type fixed, parent base_link, child caster_wheel, origin xyz=0.15 0 0.05 rpy=0 0 0, axis 0 0 1
- added joint left_wheel_joint: type continuous, parent base_link, child left_wheel, origin xyz=-0.1 0.15 0.05 rpy=-1.570796 0 0, axis 0 0 1
- added joint right_wheel_joint: type continuous, parent base_link, child right_wheel, origin xyz=-0.1 -0.15 0.05 rpy=-1.570796 0 0, axis 0 0 1
